File: Hardware/OptiComms.kicad_pcb (KiCad board)
At the start: 2 copper layers, 32 x 11 mm, 10 parts, among them J1 Conn_01x03, Q1 NPN, U1 LM393

Commit message: AC coupled test hardware
Parts:
- added C3: 1u, Capacitor_SMD:C_0603_1608Metric_Pad1.05x0.95mm_HandSolder, F.Cu at (143.8, 112.8)
- added R10: 100k, Resistor_SMD:R_0603_1608Metric_Pad1.05x0.95mm_HandSolder, F.Cu at (158.0, 111.2)
- added R6: 100k, Resistor_SMD:R_0603_1608Metric_Pad1.05x0.95mm_HandSolder, F.Cu at (149.0, 114.2)
- added R7: 102k, Resistor_SMD:R_0603_1608Metric_Pad1.05x0.95mm_HandSolder, F.Cu at (149.0, 111.2)
- added R8: 100k, Resistor_SMD:R_0603_1608Metric_Pad1.05x0.95mm_HandSolder, F.Cu at (153.5, 114.2)
- added R9: 100k, Resistor_SMD:R_0603_1608Metric_Pad1.05x0.95mm_HandSolder, F.Cu at (153.5, 111.2)
- J1: value Conn_01x03 -> Conn_01x04; footprint Connector_PinHeader_2.54mm:PinHeader_1x03_P2.54mm_Vertical -> Connector_PinHeader_2.54mm:PinHeader_1x04_P2.54mm_Vertical
Connections:
- net /OUT renamed /OUT1
- J1 pad 3: GND -> /OUT2
- U1 pad 5: (no net) -> Net-(R8-Pad2)
- U1 pad 6: (no net) -> Net-(C3-Pad2)
- U1 pad 7: (no net) -> /OUT2
Routing:
- net VCC: track 29.5 -> 63.9 mm
- net Net-(C3-Pad2): track 0.00 -> 19.3 mm
- net /OUT2: track 0.00 -> 12.5 mm
- net Net-(R8-Pad2): track 0.00 -> 8.75 mm
- net Net-(C3-Pad1): track 13.3 -> 19.1 mm
- net GND: track 6.74 -> 9.49 mm, vias 3 -> 4
Other:
- board size 32 x 11 mm -> 32 x 17 mm
- board text added: "1"
- board text added: "2"
- board text removed: "OUT"
