File: Hardware/OptiComms.sch (KiCad schematic (older format))
At the start: 10 parts, among them J1 Conn_01x03, Q1 NPN, U1 LM393

Commit message: AC coupled test hardware
Parts:
- removed J1: Conn_01x03, Connector_PinHeader_2.54mm:PinHeader_1x03_P2.54mm_Vertical, symbol Connector_Generic:Conn_01x03
- added C3: 1u, Capacitor_SMD:C_0603_1608Metric_Pad1.05x0.95mm_HandSolder, symbol Device:C
- added J1: Conn_01x04, Connector_PinHeader_2.54mm:PinHeader_1x04_P2.54mm_Vertical, symbol Connector_Generic:Conn_01x04
- added R10, R6, R8, R9: 100k, Resistor_SMD:R_0603_1608Metric_Pad1.05x0.95mm_HandSolder, symbol Device:R
- added R7: 102k, Resistor_SMD:R_0603_1608Metric_Pad1.05x0.95mm_HandSolder, symbol Device:R
- added unit 2 of U1
Connections:
- net GND: now also J1.4 (Pin_4), R7.2, R9.2
- net VCC: now also J1.1 (Pin_1), R10.1, R6.1, R8.1
- net at Q1.1 (C), R1.2, R2.2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: now also C3.1
- net OUT renamed OUT1
- net OUT1: now also J1.2 (Pin_2)
- new net: C3.2, R6.2, R7.1, U1.6 (_)
- new net: R8.2, R9.1, U1.5 (+)
- new net OUT2: J1.3 (Pin_3), R10.2, U1.7
Other:
- moved on the sheet: C1, C2, Q1, R1, R2, R3, R4, R5, U1A
